File: LED_Dimmer_12V.sch (KiCad schematic (older format))
At the start: 10 parts, among them IC1 NE555, T1 IRF610

Commit message: v1.2, THT footprints for R1 and Cs. Updated README with 3D render and picture of first populated PCB.
Parts:
- C1: value 0.1µF -> 10nF
- R1: value 10K -> 1K
Changed lines of the file:
@@
 P 5050 2650
 F 0 "R1" V 5130 2650 50  0000 C CNN
-F 1 "10K" V 5050 2650 50  0000 C CNN
+F 1 "1K" V 5050 2650 50  0000 C CNN
 F 2 "Resistors_THT:R_Axial_DIN0207_L6.3mm_D2.5mm_P2.54mm_Vertical" V 4980 2650 50  0001 C CNN
 F 3 "" H 5050 2650 50  0001 C CNN
@@
 P 4750 4050
 F 0 "C1" H 4775 4150 50  0000 L CNN
-F 1 "0.1µF" H 4775 3950 50  0000 L CNN
+F 1 "10nF" H 4775 3950 50  0000 L CNN
 F 2 "Capacitors_SMD:C_0201" H 4788 3900 50  0001 C CNN
 F 3 "" H 4750 4050 50  0001 C CNN
